File: PCB/Ganjing 75/GanJing 75.kicad_sch (KiCad schematic)
At the start: 251 parts, among them J1 1054500101, SW1 EC11, SW2 SW_Push, SW3 SW_Push, U1 USBLC6-2SC6, U2 XC6206P332MR, U3 RP2040, U4 W25Q128JVS, U5 TXS0101, Y1 12MHz

Commit message: Moving project to new PC
Parts:
- removed U3: RP2040, RP2040:RP2040-QFN-56, symbol Sleep-lib:RP2040
- added U3: RP2040, GanJing_components:RP2040-QFN-56, symbol GanJing_components:RP2040
Connections:
- net +1V1: now also U3.23 (DVDD), U3.45 (VREG_VOUT), U3.50 (DVDD)
- net +3V3: now also U3.1 (IOVDD), U3.10 (IOVDD), U3.22 (IOVDD), U3.33 (IOVDD), U3.42 (IOVDD), U3.43 (ADC_AVDD), U3.44 (VREG_VIN), U3.48 (USB_VDD), U3.49 (IOVDD)
- net COL_1: now also U3.2 (GPIO0)
- net COL_10: now also U3.12 (GPIO9)
- net COL_11: now also U3.13 (GPIO10)
- net COL_12: now also U3.14 (GPIO11)
- net COL_13: now also U3.15 (GPIO12)
- net COL_14: now also U3.16 (GPIO13)
- net COL_15: now also U3.17 (GPIO14)
- net COL_2: now also U3.3 (GPIO1)
- net COL_3: now also U3.4 (GPIO2)
- net COL_4: now also U3.5 (GPIO3)
- net COL_5: now also U3.6 (GPIO4)
- net COL_6: now also U3.7 (GPIO5)
- net COL_7: now also U3.8 (GPIO6)
- net COL_8: now also U3.9 (GPIO7)
- net COL_9: now also U3.11 (GPIO8)
- net D_R+: now also U3.47 (D+)
- net D_R-: now also U3.46 (D-)
- net GND: now also U3.19 (TESTEN), U3.57 (GND)
- net QSPI_CLK: now also U3.52 (QSPI_SCLK)
- net RGB_D0: now also U3.37 (GPIO25)
- net ROTORY_A: now also U3.32 (GPIO21)
- net ROTORY_B: now also U3.34 (GPIO22)
- net ROW_1: now also U3.18 (GPIO15)
- net ROW_2: now also U3.27 (GPIO16)
- net ROW_3: now also U3.28 (GPIO17)
- net ROW_4: now also U3.29 (GPIO18)
- net ROW_5: now also U3.30 (GPIO19)
- net ROW_6: now also U3.31 (GPIO20)
- net SCL: now also U3.36 (GPIO24)
- net SD0: now also U3.53 (QSPI_SD0)
- net SD1: now also U3.55 (QSPI_SD1)
- net SD2: now also U3.54 (QSPI_SD2)
- net SD3: now also U3.51 (QSPI_SD3)
- net SDA: now also U3.35 (GPIO23)
- net SWCLK: now also U3.24 (SWCLK)
- net SWDIO: now also U3.25 (SWDIO)
- net /CS: now also U3.56 (QSPI_SS_N)
- net /RESET: now also U3.26 (~{RUN})
- net at C13.2, Y1.3: now also U3.20 (XTAL_IN)
- net at R6.2: now also U3.21 (XTAL_OUT)
Changed lines of the file:
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@@
     (pin "2")
   )
-  (symbol (lib_id "Sleep-lib:RP2040") (at 99.06 203.2 0) (unit 1)
-    (in_bom yes) (on_board yes)
-    (property "Reference" "U3" (id 0) (at 81.28 153.67 0)
-      (effects (font (size 1.27 1.27)) (justify left))
-    )
-    (property "Value" "RP2040" (id 1) (at 81.28 250.19 0)
-      (effects (font (size 1.27 1.27)) (justify left))
-    )
-    (property "Footprint" "RP2040:RP2040-QFN-56" (id 2) (at 78.74 140.97 0)
-      (effects (font (size 1.27 1.27)) (justify left bottom) hide)
-    )
-    (property "Datasheet" "https://datasheets.raspberrypi.com/rp2040/rp2040-datasheet.pdf" (id 3) (at 78.74 140.97 0)
-      (effects (font (size 1.27 1.27)) (justify left bottom) hide)
-    )
-    (property "JLC P#" "C2040" (id 4) (at 99.06 203.2 0)
-      (effects (font (size 1.27 1.27)) hide)
-    )
-    (pin "1")
-    (pin "10")
-    (pin "11")
-    (pin "12")
-    (pin "13")
-    (pin "14")
-    (pin "15")
-    (pin "16")
-    (pin "17")
-    (pin "18")
-    (pin "19")
-    (pin "2")
-    (pin "20")
-    (pin "21")
-    (pin "22")
-    (pin "23")
-    (pin "24")
-    (pin "25")
-    (pin "26")
-    (pin "27")
-    (pin "28")
-    (pin "29")
-    (pin "3")
-    (pin "30")
-    (pin "31")
-    (pin "32")
-    (pin "33")
-    (pin "34")
-    (pin "35")
-    (pin "36")
-    (pin "37")
-    (pin "38")
-    (pin "39")
-    (pin "4")
-    (pin "40")
-    (pin "41")
-    (pin "42")
-    (pin "43")
-    (pin "44")
-    (pin "45")
-    (pin "46")
-    (pin "47")
-    (pin "48")
-    (pin "49")
-    (pin "5")
-    (pin "50")
-    (pin "51")
-    (pin "52")
-    (pin "53")
-    (pin "54")
-    (pin "55")
-    (pin "56")
-    (pin "57")
-    (pin "6")
-    (pin "7")
-    (pin "8")
-    (pin "9")
-  )
   (symbol (lib_id "Diode:1N4148WS") (at 290.83 88.9 90) (unit 1)
     (in_bom yes) (on_board yes) (fields_autoplaced)
@@
     (pin "2")
   )
+  (symbol (lib_id "GanJing_components:RP2040") (at 99.06 203.2 0) (unit 1)
+    (in_bom yes) (on_board yes)
+    (property "Reference" "U3" (id 0) (at 81.28 153.67 0)
+      (effects (font (size 1.27 1.27)) (justify left))
+    )
+    (property "Value" "RP2040" (id 1) (at 95.25 203.2 0)
+      (effects (font (size 1.27 1.27)) (justify left))
+    )
+    (property "Footprint" "GanJing_components:RP2040-QFN-56" (id 2) (at 78.74 140.97 0)
+      (effects (font (size 1.27 1.27)) (justify left bottom) hide)
+    )
+    (property "Datasheet" "https://datasheets.raspberrypi.com/rp2040/rp2040-datasheet.pdf" (id 3) (at 78.74 140.97 0)
+      (effects (font (size 1.27 1.27)) (justify left bottom) hide)
+    )
+    (pin "1")
+    (pin "10")
+    (pin "11")
+    (pin "12")
+    (pin "13")
+    (pin "14")
+    (pin "15")
+    (pin "16")
+    (pin "17")
+    (pin "18")
+    (pin "19")
+    (pin "2")
+    (pin "20")
+    (pin "21")
+    (pin "22")
+    (pin "23")
+    (pin "24")
+    (pin "25")
+    (pin "26")
+    (pin "27")
+    (pin "28")
+    (pin "29")
+    (pin "3")
+    (pin "30")
+    (pin "31")
+    (pin "32")
+    (pin "33")
+    (pin "34")
+    (pin "35")
+    (pin "36")
+    (pin "37")
+    (pin "38")
+    (pin "39")
+    (pin "4")
+    (pin "40")
+    (pin "41")
+    (pin "42")
+    (pin "43")
+    (pin "44")
+    (pin "45")
+    (pin "46")
+    (pin "47")
+    (pin "48")
+    (pin "49")
+    (pin "5")
+    (pin "50")
+    (pin "51")
+    (pin "52")
+    (pin "53")
+    (pin "54")
+    (pin "55")
+    (pin "56")
+    (pin "57")
+    (pin "6")
+    (pin "7")
+    (pin "8")
+    (pin "9")
+  )
   (symbol (lib_id "GanJing_components:MX_1u_no_LED") (at 344.17 41.91 0) (unit 1)
     (in_bom yes) (on_board yes)
@@
       (reference "U2") (unit 1) (value "XC6206P332MR") (footprint "GanJing_components:SOT-23-3")
     )
-    (path "/7eb525f4-c9fd-4c61-9b22-fdd518f97c1c"
-      (reference "U3") (unit 1) (value "RP2040") (footprint "RP2040:RP2040-QFN-56")
+    (path "/85413da7-5225-4bf6-a3cf-6c3b1329f212"
+      (reference "U3") (unit 1) (value "RP2040") (footprint "GanJing_components:RP2040-QFN-56")
     )
     (path "/45fe62ec-79f8-462d-b42b-4660408ea65a"
